File: SmartCard.kicad_sch (KiCad schematic)
At the start: 12 parts, among them IC1 BQ298009RUGR, Q1 EFC3J018NUZTDG, U1 BQ51050BRHL, U2 NRF54L15-QFAA-R

Commit message: Refactor KiCad schematic symbols & positions
Adjust schematic symbols and component placements in SmartCard.kicad_sch and update project metadata in SmartCard.kicad_pro. Changes include repositioning pins and boxes for multiple components (e.g. U1 / BQ51050BRHL), replacing/respecifying symbol types (R -> FerriteBead, new L/inductor symbols), reorganizing the NRF54L15 part definition and properties, and updating used_designators. Also add a timestamped backup archive SmartCard-backups/SmartCard-2026-05-06_220005.zip.
Parts:
- added C10, C12: 2.2uF, symbol Device:C_Small
- added C11: 3.9pF, symbol Device:C_Small
- added C13, C17, C31, C40: 22nF, symbol Device:C_Small
- added C14, C18, C28, C30, C38, C9: 10nF, symbol Device:C_Small
- added C15, C22, C24, C34, C35, C7: 10uF, symbol Device:C_Small
- added C16, C21, C32, C33: 0.47uF, symbol Device:C_Small
- added C19: 2.5nF, symbol Device:C_Small
- added C20: 253nF, symbol Device:C_Small
- added C23, C25, C3, C4, C41, C42, C5, C6: 0.1uF, symbol Device:C_Small
- added C26: 270pF, symbol Device:C_Small
- added C29, C36, C37: 100nF, symbol Device:C_Small
- added C39: 2.7nF, symbol Device:C_Small
- added C8: 2.2nF, symbol Device:C_Small
- added FB1: 120, symbol Device:FerriteBead
- added IC2: BQ25170DSGR, SON50P200X200X80-9N, symbol SamacSys_Parts:BQ25170DSGR
- added IC3: BQ51003YFPT, BGA28C40P4X7_188X301X50, symbol SamacSys_Parts:BQ51003YFPT
- added L1: 4.7uF, symbol Device:L
- added L2: RX COIL, symbol Device:L
- added R10, R14: 200, symbol Device:R
- added R11: ROS, symbol Device:R
- added R12, R13, R15: 6.2k, symbol Device:R
- added R16, R8: 10k, symbol Device:R
- added R7: 1k, symbol Device:R
- added R9: 60.4k, symbol Device:R
Connections:
- net GND: now also U1.1 (PGND), U1.11 (EN2), U1.20 (PGND), U1.21 (PGND), U1.9 (AD), U2.44 (VSS), U2.49 (VSS__1), C10.2, C11.2, C12.2, C15.2, C22.2, C23.2, C24.2, C25.2, C3.2, C34.2, C35.2, C4.2, C41.2, C42.2, C5.2, C6.2, C7.2, C8.2, C9.2, IC3.A1 (PGND), IC3.A2 (PGND), IC3.A3 (PGND), IC3.A4 (PGND), IC3.G2 (EN2), IC3.G3 (EN1), IC3.G4 (AD), R10.2, R14.2, R16.2, R8.2, R9.2
- net VBUS: now also U1.4 (BAT), C15.1, C23.1
- net at U1.10 (TERM): now also R9.1
- net at U1.12 (ILIM): now also R12.1
- net at U1.13 (TS/CTRL): now also R8.1
- net at U1.14 (FOD): now also R10.1, R11.2, R12.2
- net at U1.15 (COMM2): now also C17.1
- net at U1.16 (CLAMP2): now also C16.1
- net at U1.17 (BOOT2): now also C18.1
- net at U1.18 (RECT): now also C22.1, C24.1, C25.1, R11.1
- net at U1.19 (AC2): now also C16.2, C17.2, C18.2, C19.1
- net at U1.2 (AC1): now also C13.2, C14.2, C19.2, C20.2, C21.2
- net at U1.3 (BOOT1): now also C14.1
- net at U1.5 (CLAMP1): now also C21.1
- net at U1.6 (COMM1): now also C13.1
- net at U2.10 (VDD): now also U2.22 (VDD__1), U2.36 (VDD__2), U2.47 (VDD__3), U2.48 (VDD__4), C3.1, C4.1, C5.1, C6.1, C7.1
- net XL1: now reaches U2.23 (P0.00)
- net XL2: now reaches U2.24 (P0.01)
- net SWDIO: now reaches U2.25 (SWDIO)
- net SWDCLK: now reaches U2.26 (SWDCLK)
- net at U2.30 (~{RESET}): now also C11.1, R7.1
- net at U2.33 (DECRF): now also U2.43 (DECA), C10.1, C8.1, C9.1, FB1.2
- net XC1: now reaches U2.34 (XC1)
- net XC2: now reaches U2.35 (XC2)
- net at U2.45 (DECD): now also C12.1, FB1.1, L1.1
- net at U2.46 (DCC): now also L1.2
- new net: C26.1, C28.1, C29.2, C33.1, C36.2, C37.2, C38.2, C39.1, C40.1, IC3.B3 (AC1), IC3.B4 (AC1)
- new net: C28.2, IC3.C4 (BOOT1)
- new net: C34.1, C42.1, IC3.C2 (RECT), IC3.C3 (RECT), R15.1
- new net: C40.2, IC3.E4 (COMM1)
- new net: C26.2, C30.1, C31.1, C32.1, C39.2, IC3.B1 (AC2), IC3.B2 (AC2), L2.1
- new net: C30.2, IC3.C1 (BOOT2)
- new net: C35.1, C41.1, IC3.D1 (OUT), IC3.D2 (OUT), IC3.D3 (OUT), IC3.D4 (OUT), IC3.F2 (FOD), R13.2, R14.1, R15.2
- new net: C31.2, IC3.E1 (COMM2)
- new net: C33.2, IC3.E2 (CLAMP2)
- new net: C32.2, IC3.E3 (CLAMP1)
- new net: IC3.F1 (TS-CTRL), R16.1
- new net: IC3.G1 (ILIM), R13.1
- new net: C29.1, C36.1, C37.1, C38.1, L2.2
- new net RESET: R7.2
- no-connect marks 0 -> 2
Other:
- note added: "2.97nF"
- note added: "~304nF"
- moved on the sheet: U1, U2

Commit message: Update KiCad schematic symbols & add backups
Add three SmartCard backup zip files and update the KiCad project files. SmartCard.kicad_sch: introduce new/updated library symbols (Abracon AMCA31 transducer, ABM11W oscillator replacing a prior part, ECS 32.768kHz crystal), adjust properties (reference, value, footprint, datasheet, manufacturer, pin names), add VDD power symbol, and relocate/update many symbol positions and junctions. SmartCard.kicad_pro: simplify used_designators entry to "C44-46,Y2,E1". These changes ensure correct component metadata and footprints in the schematic.
Parts:
- added C27, C43: 1uF, symbol Device:C_Small
- added C44, C45, C46: 8pF, symbol Device:C_Small
- added E1: AMCA31-2R450G-S1F-T3, AMCA31-2R450G-S1F-T3:XDCR_AMCA31-2R450G-S1F-T3, symbol AMCA31-2R450G-S1F-T3:AMCA31-2R450G-S1F-T3
- added R17: 20k, symbol Device:R
- added R18, R20: 7.5k, symbol Device:R
- added R19: 27k, symbol Device:R
- added Y1: ABM11W-25.0000MHZ-7-D1X-T3, ABM11W300000MHZ4B1UT3, symbol SamacSys_Parts:ABM11W-25.0000MHZ-7-D1X-T3
- added Y2: ECS-.327-7-12-TR, ECS327712TR, symbol SamacSys_Parts:ECS-.327-7-12-TR
- C32, C33: value 0.47uF -> 470nF
- R13: value 6.2k -> 2.43k
- R15: value 6.2k -> ROS2
Connections:
- net GND: now also IC2.4 (GND), IC2.9 (EP), C27.2, C43.2, R18.1, R19.1, R20.1
- net VBUS: now also C35.1, C41.1, IC2.1 (IN), IC3.D1 (OUT), IC3.D2 (OUT), IC3.D3 (OUT), IC3.D4 (OUT), C27.1, R17.1; no longer Q1.1 (SOURCE1), Q1.3 (SOURCE1), R2.1, R3.1
- net at IC2.2 (ISET): now also R18.2
- net at IC2.3 (TS): now also R20.2
- net at IC2.7 (VSET): now also R19.2
- net VDD: now reaches IC2.8 (OUT)
- net VDD: now also Q1.1 (SOURCE1), Q1.3 (SOURCE1), R2.1, R3.1, C43.1
- new net: IC3.F2 (FOD), R13.2, R14.1, R15.2, R17.2
- new net: C46.1, Y1.1 (X1)
- new net: C44.1, Y1.2 (GND_1)
- no-connect marks 2 -> 4
Other:
- moved on the sheet: C1, C10, C11, C12, C2, C26, C28, C29, C3, C30, C31, C32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

Commit message: Update KiCad prefs, board rules, schematic
Add backup zips and update KiCad project files: expand net inspector column settings in SmartCard.kicad_prl; add comprehensive design_settings (DRC/rules, teardrops, track/tuning defaults, via/zones) and clear used_designators in SmartCard.kicad_pro; apply many edits to SmartCard.kicad_sch (add BQ25100 symbol, adjust text/footprint labels, add text_box, reposition junctions/wires, add/remove junctions and wire segments, update UUIDs). These changes capture project preferences, board DRC defaults, and schematic layout/connection fixes.
Parts:
- removed C36, C37: 100nF, symbol Device:C_Small
- removed R13: 2.43k, symbol Device:R
- removed R14: 200, symbol Device:R
- removed R15: ROS2, symbol Device:R
- added C47: 1uF, symbol Device:C_Small
- added C48: 100nF, symbol Device:C_Small
- added IC4: BQ25100YFPR, BGA6C40P2X3_88X158X50, symbol SamacSys_Parts:BQ25100YFPR
- added R21: 7.5k, symbol Device:R
- added R22: 6k, symbol Device:R
- added R23: 3.4k, symbol Device:R
- added R24: 196, symbol Device:R
- added R25: 6.34k, symbol Device:R
- C26: value 270pF -> 47pF
- C39: value 2.7nF -> 1.3nF
Connections:
- net GND: now also C47.2, C48.1, IC4.C2 (VSS), R21.2, R22.1, R23.1, R24.2
- net VBUS: now also C48.2, IC4.A2 (IN); no longer R17.1
- net VDD: now also C47.1, IC4.A1 (OUT)
- net RECT: now reaches C34.1, C42.1, IC3.C2 (RECT), IC3.C3 (RECT)
- net RECT: now also R17.1
- net FOD: now reaches IC3.F2 (FOD), R17.2
- net FOD: now also R24.1, R25.1
- net ILIM: now reaches IC3.G1 (ILIM)
- net ILIM: now also R25.2
- new net: IC4.B1 (TS), R21.1
- new net: IC4.B2 (ISET), R23.2
- new net: IC4.C1 (PRETERM), R22.2
Other:
- note added: "C1"
- note added: "C2"
- note added: "~1.349nF"
- note added: "~111.1nF"
- note removed: "2.97nF"
- note removed: "~304nF"
- moved on the sheet: C27, C43, IC2, R18, R19, R20
