File: SmartCard.kicad_sch (KiCad schematic)
At the start: 81 parts, among them IC1 BQ298009RUGR, IC2 BQ25170DSGR, IC3 BQ51003YFPT, IC4 BQ25100YFPR, Q1 EFC3J018NUZTDG, U1 BQ51050BRHL, U2 NRF54L15-QFAA-R, Y1 ABM11W-25.0000MHZ-7-D1X-T3, Y2 ECS-.327-7-12-TR

Commit message: finished v0.1 shematic
Parts:
- removed C13, C17: 22nF, symbol Device:C_Small
- removed C14, C18: 10nF, symbol Device:C_Small
- removed C15, C22, C24: 10uF, symbol Device:C_Small
- removed C16, C21: 0.47uF, symbol Device:C_Small
- removed C19: 2.5nF, symbol Device:C_Small
- removed C20: 253nF, symbol Device:C_Small
- removed C23: 0.1uF, symbol Device:C_Small
- removed C27, C43: 1uF, symbol Device:C_Small
- removed IC2: BQ25170DSGR, SON50P200X200X80-9N, symbol SamacSys_Parts:BQ25170DSGR
- removed R10: 200, symbol Device:R
- removed R11: ROS, symbol Device:R
- removed R12: 6.2k, symbol Device:R
- removed R18, R20: 7.5k, symbol Device:R
- removed R19: 27k, symbol Device:R
- removed R5: 100, symbol Device:R
- removed R8: 10k, symbol Device:R
- removed R9: 60.4k, symbol Device:R
- removed U1: BQ51050BRHL, Package_DFN_QFN:Texas_VQFN-RHL-20, symbol Battery_Management:BQ51050BRHL
- added C31, C36: 1.5pF, Capacitor_SMD:C_0201_0603Metric, symbol Device:C_Small
- added C33: 2.0pF, Capacitor_SMD:C_0201_0603Metric, symbol Device:C_Small
- added C34: 4.7uF, Capacitor_SMD:C_0603_1608Metric, symbol Device:C_Small
- added C35: 0.3pF, Capacitor_SMD:C_0201_0603Metric, symbol Device:C_Small
- added C38: DNP, Capacitor_SMD:C_0201_0603Metric, symbol Device:C_Small
- added C39: 10uF, Capacitor_SMD:C_0603_1608Metric, symbol Device:C_Small
- added L3: 2.7nH, Inductor_SMD:L_0201_0603Metric, symbol Device:L
- added L4, L5: 3.5nH, Inductor_SMD:L_0201_0603Metric, symbol Device:L
- added L6: 3.9nH, Inductor_SMD:L_0201_0603Metric, symbol Device:L
- added L7: 2.2uH, Inductor_SMD:L_0603_1608Metric, symbol Device:L
- added U2: TPS62840YBGR, SamacSys_Parts:TPS62840YBGR, symbol TPS62840YBGR:TPS62840YBGR
- C1: renamed from C10; footprint (none) -> Capacitor_SMD:C_0402_1005Metric
- C10: renamed from C30; footprint (none) -> Capacitor_SMD:C_0402_1005Metric
- C11: renamed from C31; footprint (none) -> Capacitor_SMD:C_0402_1005Metric
- C12: renamed from C32; footprint (none) -> Capacitor_SMD:C_0402_1005Metric
- C13: renamed from C33; footprint (none) -> Capacitor_SMD:C_0402_1005Metric
- C14: renamed from C39; footprint (none) -> Capacitor_SMD:C_0603_1608Metric
- C15: renamed from C11; footprint (none) -> Capacitor_SMD:C_0402_1005Metric
- C16: renamed from C3; footprint (none) -> Capacitor_SMD:C_0402_1005Metric
- C17: renamed from C35; footprint (none) -> Capacitor_SMD:C_0603_1608Metric
- C18: renamed from C34; footprint (none) -> Capacitor_SMD:C_0603_1608Metric
- C19: renamed from C4; footprint (none) -> Capacitor_SMD:C_0402_1005Metric
- C2: renamed from C9; footprint (none) -> Capacitor_SMD:C_0402_1005Metric
- C20: renamed from C41; footprint (none) -> Capacitor_SMD:C_0402_1005Metric
- C21: renamed from C42; footprint (none) -> Capacitor_SMD:C_0402_1005Metric
- C22: renamed from C5; footprint (none) -> Capacitor_SMD:C_0402_1005Metric
- C23: renamed from C46; footprint (none) -> Capacitor_SMD:C_0402_1005Metric
- C24: renamed from C6; footprint (none) -> Capacitor_SMD:C_0402_1005Metric
- C25: value 0.1uF -> 8pF; footprint (none) -> Capacitor_SMD:C_0402_1005Metric
- C26: renamed from C7; footprint (none) -> Capacitor_SMD:C_0603_1608Metric
- C27: renamed from C48; value 100nF -> 0.1uF; footprint (none) -> Capacitor_SMD:C_0402_1005Metric
- C28: renamed from C45; footprint (none) -> Capacitor_SMD:C_0402_1005Metric
- C29: renamed from C44; footprint (none) -> Capacitor_SMD:C_0402_1005Metric
- C3: renamed from C12; footprint (none) -> Capacitor_SMD:C_0402_1005Metric
- C30: renamed from C47; footprint (none) -> Capacitor_SMD:C_0603_1608Metric
- C32: renamed from C1; footprint (none) -> Capacitor_SMD:C_0402_1005Metric
- C37: renamed from C2; footprint (none) -> Capacitor_SMD:C_0402_1005Metric
- C4: renamed from C8; footprint (none) -> Capacitor_SMD:C_0402_1005Metric
- C5: renamed from C38; footprint (none) -> Capacitor_SMD:C_0603_1608Metric
- C6: renamed from C29; footprint (none) -> Capacitor_SMD:C_0603_1608Metric
- C7: renamed from C26; footprint (none) -> Capacitor_SMD:C_0603_1608Metric
- C8: renamed from C40; footprint (none) -> Capacitor_SMD:C_0402_1005Metric
- C9: renamed from C28; footprint (none) -> Capacitor_SMD:C_0402_1005Metric
- E1: footprint AMCA31-2R450G-S1F-T3:XDCR_AMCA31-2R450G-S1F-T3 -> SamacSys_Parts:XDCR_AMCA31-2R450G-S1F-T3
- FB1: footprint (none) -> Inductor_SMD:L_0402_1005Metric
- IC1: renamed from IC3; footprint BGA28C40P4X7_188X301X50 -> SamacSys_Parts:BGA28C40P4X7_188X301X50
- IC2: renamed from IC4; footprint BGA6C40P2X3_88X158X50 -> SamacSys_Parts:BGA6C40P2X3_88X158X50
- IC3: renamed from IC1; footprint BQ298009RUGR -> SamacSys_Parts:BQ298009RUGR
- L1: value 4.7uF -> 4.7uH; footprint (none) -> Inductor_SMD:L_0603_1608Metric
- L2: footprint (none) -> Inductor_SMD:L_1206_3216Metric_Pad1.22x1.90mm_HandSolder
- Q1: footprint EFC3J018NUZTDG -> SamacSys_Parts:EFC3J018NUZTDG
- R1: renamed from R25; footprint (none) -> Resistor_SMD:R_0402_1005Metric
- R10: renamed from R6; footprint (none) -> Resistor_SMD:R_0603_1608Metric
- R11: renamed from R2; footprint (none) -> Resistor_SMD:R_0402_1005Metric
- R12: renamed from R4; value 5M -> 4.7M; footprint (none) -> Resistor_SMD:R_0402_1005Metric
- R14: renamed from R1; footprint (none) -> Resistor_SMD:R_0402_1005Metric
- R2: renamed from R24; footprint (none) -> Resistor_SMD:R_0402_1005Metric
- R3: renamed from R17; footprint (none) -> Resistor_SMD:R_0402_1005Metric
- R4: renamed from R7; footprint (none) -> Resistor_SMD:R_0402_1005Metric
- R5: renamed from R16; footprint (none) -> Resistor_SMD:R_0402_1005Metric
- R6: renamed from R23; footprint (none) -> Resistor_SMD:R_0402_1005Metric
- R7: renamed from R22; footprint (none) -> Resistor_SMD:R_0402_1005Metric
- R8: renamed from R21; footprint (none) -> Resistor_SMD:R_0402_1005Metric
- R9: renamed from R3; footprint (none) -> Resistor_SMD:R_0402_1005Metric
- U1: renamed from U2; footprint NRF54L15-QFAA-R:QFN40P600X600X90-49N -> SamacSys_Parts:QFN40P600X600X90-49N
- Y1: footprint ABM11W300000MHZ4B1UT3 -> SamacSys_Parts:ABM11W300000MHZ4B1UT3
- Y2: footprint ECS327712TR -> SamacSys_Parts:ECS327712TR
Connections:
- net CTR: now also C37.1, IC3.5 (CTR), R12.1
- net GND: now also C23.2, C28.2, C29.2, U1.32 (VSS_PA), Y1.2 (GND_1), Y1.4 (GND_2), C31.1, C33.1, C34.2, C35.1, C36.1, C38.1, C39.2, U2.A1 (GND), U2.C2 (VSET)
- net VDD: now also C34.1, U2.B1 (VIN), U2.C1 (EN)
- net XC1: now also C23.1, Y1.1 (X1)
- net XC2: now also C29.1, Y1.3 (X2)
- net XL1: now also C25.1, U1.1 (P1.00/XL1), Y2.; no longer U1.23 (P0.00)
- net XL2: now also C28.1, U1.2 (P1.01/XL2), Y2.2 (OUT/IN); no longer U1.24 (P0.01)
- net +1V8: now reaches C16.1, C19.1, C22.1, C24.1, C26.1, U1.10 (VDD), U1.22 (VDD__1), U1.36 (VDD__2), U1.47 (VDD__3), U1.48 (VDD__4)
- net +1V8: now also C39.1, L7.2, U2.A2 (VOS)
- net at E1.1: now also C38.2, L6.2
- net ANT: now reaches U1.31 (ANT)
- net ANT: now also L3.1
- new net: C33.2, L4.2, L5.1
- new net: C35.2, C36.2, L5.2, L6.1
- new net: L7.1, U2.B2 (SW)
- new net: C31.2, L3.2, L4.1
- no-connect marks 4 -> 30
Other:
- note added: "1v8 Buck Converter"
- note added: "RF Matching Network"
- note added: "To Bottom Layer"
- note added: "To PIN 49"
- note added: "Wireless Power and Battery Charging"
- note added: "nRF54L15"
- moved on the sheet: C1, C10, C11, C12, C13, C14, C15, C16, C17, C18, C19, C2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

Commit message: Populate SmartCard PCB and add test points
Adds the full KiCad PCB implementation from the previously minimal board file, including footprints, board outline, and RF/power sections. Updates the schematic with test point symbols/instances (TP1-TP4) and related power labels, and refreshes project settings (.kicad_pro/.kicad_prl) for routing, DRC, and zone defaults to match the expanded design.
Parts:
- added TP1: GND, symbol Connector:TestPoint
- added TP2: 1V8, symbol Connector:TestPoint
- added TP3: BATT, symbol Connector:TestPoint
- added TP4: VDD, symbol Connector:TestPoint
Connections:
- net +1V8: now also TP2.1
- net +BATT: now also TP3.1
- net GND: now also TP1.1
- net VDD: now also TP4.1

Commit message: mostly done just a little more work
Parts:
- removed C37: 1uF, Capacitor_SMD:C_0402_1005Metric, symbol Device:C_Small
- removed IC1: BQ51003YFPT, SamacSys_Parts:BGA28C40P4X7_188X301X50, symbol SamacSys_Parts:BQ51003YFPT
- removed R12: 4.7M, Resistor_SMD:R_0402_1005Metric, symbol Device:R
- added IC1: BQ51013BRHLR, Package_DFN_QFN:Texas_VQFN-RHL-20, symbol SamacSys_Parts:BQ51013BRHLR
- added J1: Conn_01x05, Connector_PinHeader_2.54mm:PinHeader_1x05_P2.54mm_Vertical, symbol Connector_Generic:Conn_01x05
- added TP5: VBUS, TestPoint:TestPoint_Pad_2.0x2.0mm, symbol Connector:TestPoint
- C1, C3: DPN (none) -> 490-10450-1-ND; MPN (none) -> GRM155D80J225ME95D
- C10, C2, C5, C9: DPN (none) -> 490-4516-1-ND; MPN (none) -> GRM155R71H103KA88D
- C11, C8: DPN (none) -> 490-3884-1-ND; MPN (none) -> GRM155R71H223KA12D
- C12, C13: DPN (none) -> 445-8020-1-ND; MPN (none) -> C1005X5R1E474K050BB
- C14: value 1.3nF -> 1nF; DPN (none) -> 490-1303-1-ND; MPN (none) -> GRM155R71H102KA01D
- C15: DPN (none) -> 490-6239-1-ND; MPN (none) -> GRM1555C1H3R9BA01D
- C16, C19, C20, C21, C22, C24, C27, C32, C6: DPN (none) -> 490-10700-1-ND; MPN (none) -> GRM155R71H104KE14D
- C17, C18, C26, C39: DPN (none) -> 490-12323-1-ND; MPN (none) -> GRT188R61E106ME13D
- C23, C25, C28, C29: DPN (none) -> 490-11238-1-ND; MPN (none) -> GJM1555C1H8R0BB01D
- C30: DPN (none) -> 587-2477-1-ND; MPN (none) -> EMK105BJ105KV-F
- C31, C36: DPN (none) -> 490-11176-1-ND; MPN (none) -> GJM0335C1E1R5WB01D
- C33: DPN (none) -> 490-GRM0335C1H2R0WA01DCT-ND; MPN (none) -> GRM0335C1H2R0WA01D
- C34: DPN (none) -> 4713-GMC10X5R475K10NTCT-ND; MPN (none) -> GMC10X5R475K10NT
- C35: DPN (none) -> 490-17810-1-ND; MPN (none) -> GRM0335C1ER30WA01D
- C38: MPN (none) -> DNP; now not fitted
- C4: DPN (none) -> 490-3256-1-ND; MPN (none) -> GRM155R71C223KA01D
- C7: value 47pF -> 330pF; DPN (none) -> 490-3247-1-ND; MPN (none) -> GRM155R71H331KA01D
- E1: DPN (none) -> 535-14095-1-ND; MPN (none) -> AMCA31-2R450G-S1F-T3
- FB1: DPN (none) -> 1934-1366-1-ND; MPN (none) -> 2504021217Y0
- IC2: DPN (none) -> 296-39931-1-ND; MPN (none) -> BQ25100YFPR
- IC3: DPN (none) -> 296-BQ298009RUGRCT-ND; MPN (none) -> BQ298009RUGR
- L1: DPN (none) -> 445-MLZ1608CWC4R7MTD25CT-ND; MPN (none) -> MLZ1608CWC4R7MTD25
- L2: footprint Inductor_SMD:L_1206_3216Metric_Pad1.22x1.90mm_HandSolder -> Inductor_SMD:L_1812_4532Metric_Pad1.30x3.40mm_HandSolder; DPN (none) -> 445-16093-ND; MPN (none) -> WR444030-16F3-G
- L3: DPN (none) -> 490-13909-1-ND; MPN (none) -> LQP03HQ2N7B02D
- L4, L5: DPN (none) -> 490-13925-1-ND; MPN (none) -> LQP03HQ3N5B02D
- L6: DPN (none) -> 490-14982-1-ND; MPN (none) -> LQP03TQ3N9B02D
- L7: DPN (none) -> 490-14478-1-ND; MPN (none) -> LQM18PN2R2MGHD
- Q1: DPN (none) -> 488-EFC3J018NUZTDGCT-ND; MPN (none) -> EFC3J018NUZTDG
- R1: DPN (none) -> YAG3218CT-ND; MPN (none) -> RC0402FR-076K34L
- R10: value 50m -> 100m; footprint Resistor_SMD:R_0603_1608Metric -> Resistor_SMD:R_0805_2012Metric; DPN (none) -> RL12S.10FCT-ND; MPN (none) -> RL1220S-R10-F
- R11: DPN (none) -> 311-20LRCT-ND; MPN (none) -> RC0402FR-0720RL
- R13: renamed from R14; DPN (none) -> 311-20.0KLRCT-ND; MPN (none) -> RC0402FR-0720KL
- R2: DPN (none) -> 541-196LCT-ND; MPN (none) -> CRCW0402196RFKED
- R3: DPN (none) -> 311-20.0KLRCT-ND; MPN (none) -> RC0402FR-0720KL
- R4: DPN (none) -> 311-1.00KLRCT-ND; MPN (none) -> RC0402FR-071KL
- R5: DPN (none) -> 311-10.0KLRCT-ND; MPN (none) -> RC0402FR-0710KL
- R6: DPN (none) -> YAG3149CT-ND; MPN (none) -> RC0402FR-073K4L
- R7: value 6k -> 6.04k; DPN (none) -> YAG2293CT-ND; MPN (none) -> RC0402FR-076K04L
- R8: DPN (none) -> 311-7.50KLRCT-ND; MPN (none) -> RC0402FR-077K5L
- R9: DPN (none) -> 311-300LRCT-ND; MPN (none) -> RC0402FR-07300RL
- TP1, TP3: footprint (none) -> TestPoint:TestPoint_Pad_2.0x2.0mm; now not fitted; now left out of the parts list
- TP2, TP4: footprint (none) -> TestPoint:TestPoint_Pad_2.0x2.0mm; now left out of the parts list
- U1: DPN (none) -> 4823-NRF54L15-QFAA-RCT-ND; MPN (none) -> NRF54L15-QFAA-R
- U2: DPN (none) -> 296-TPS62840YBGRCT-ND; MPN (none) -> TPS62840YBGR
- Y1: value ABM11W-25.0000MHZ-7-D1X-T3 -> 32MHz; DPN (none) -> 535-13898-1-ND; MPN (none) -> ABM11W-32.0000MHZ-7-D1X-T3
- Y2: DPN (none) -> 50-ECS-.327-7-12-TRCT-ND; MPN (none) -> ECS-.327-7-12-TR
Connections:
- net CTR is gone; now on net -BATT: IC3.5 (CTR)
- net FOD: now also IC1.14 (FOD)
- net GND: now also IC1.1 (PGND), IC1.11 (EN2), IC1.20 (PGND), IC1.21 (EP), IC1.9 (AD), J1.1 (Pin_1)
- net ILIM: now also IC1.12 (ILIM)
- net RECT: now also IC1.18 (RECT)
- net RESET: now also J1.4 (Pin_4)
- net SWDCLK: now also J1.3 (Pin_3)
- net SWDIO: now also J1.2 (Pin_2)
- net VBUS: now also IC1.4 (OUT), TP5.1
- net VDD: now also J1.5 (Pin_5)
- net XL1: now also Y2.1; no longer Y2.
- net at C13.1, C14.1, C5.2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: now also IC1.2 (AC1)
- net at C9.2: now also IC1.3 (BOOT1)
- net at C8.2: now also IC1.6 (COMM1)
- net at C10.1, C11.1, C12.1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: now also IC1.19 (AC2)
- net at C10.2: now also IC1.17 (BOOT2)
- net at C11.2: now also IC1.15 (COMM2)
- net at C13.2: now also IC1.5 (CLAMP1)
- net at C12.2: now also IC1.16 (CLAMP2)
- net at R5.1: now also IC1.13 (TS/CTRL)
- net EN1: now reaches U1.13 (P2.02)
- net EN1: now also IC1.10 (EN1)
- no-connect marks 30 -> 29
Other:
- moved on the sheet: C32, C34, C39, L7, R10, TP2, TP4, U2

Commit message: mostly finished
Other:
- note added: "Smart Card"
- company: (none) -> Serious Engineering
Changed lines of the file:
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@@
 	(title_block
 		(title "Smart Card")
-		(date "2026-08-17")
+		(date "2026-08-25")
 		(rev "2")
+		(company "Serious Engineering")
 	)
 	(rectangle
@@
 			)
 		)
+	)
+	(text "Smart Card"
+		(exclude_from_sim no)
+		(at 327.914 260.35 0)
+		(effects
+			(font
+				(size 6.35 6.35)
+				(bold yes)
+			)
+		)

Commit message: fixed schematic for v2 fixing bat management
still need to do layout
Parts:
- C7: value 330pF -> 100pF
Connections:
- net +BATT: now also R11.1, R9.1; no longer R13.1
- net -BATT: now also C32.2, IC3.3 (VSS), R10.1; no longer IC3.4 (CS), IC3.5 (CTR), R10.2
- net GND: now also IC3.4 (CS), IC3.5 (CTR), R10.2; no longer C32.2, IC3.3 (VSS), R10.1
- net VDD: now also R13.1; no longer R11.1, R9.1
- net at Q1.2 (GATE1): now also IC3.7 (DSG); no longer IC3.8 (CHG)
- net at Q1.5 (GATE2): now also IC3.8 (CHG); no longer IC3.7 (DSG)
Other:
- note added: "~1.11nF"
- note added: "~110nF"
- note removed: "~1.349nF"
- note removed: "~111.1nF"
