File: SmartCard.kicad_sch (KiCad schematic)
At the start: 73 parts, among them IC1 BQ51013BRHLR, IC2 BQ25100YFPR, IC3 BQ298009RUGR, J1 Conn_01x05, Q1 EFC3J018NUZTDG, U1 NRF54L15-QFAA-R, U2 TPS62840YBGR, Y1 32MHz, Y2 ECS-.327-7-12-TR

Commit message: finished pack swap
Connections:
- net GND: now also IC1.10 (EN1)
- net EN1: no longer names the net of U1.13 (P2.02)
- net EN1: no longer IC1.10 (EN1)
- no-connect marks 29 -> 30
Changed lines of the file:
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@@
 	)
 	(junction
+		(at 147.32 95.25)
+		(diameter 0)
+		(color 0 0 0 0)
+	)
+	(junction
 		(at 48.26 186.69)
 		(diameter 0)
@@
 	)
 	(no_connect
+		(at 129.54 220.98)
+	)
+	(no_connect
 		(at 63.5 205.74)
 	)
@@
 	(wire
 		(pts
+			(xy 147.32 92.71) (xy 147.32 95.25)
+		)
+		(stroke
+			(width 0)
+			(type default)
+		)
+	)
+	(wire
+		(pts
 			(xy 161.29 203.2) (xy 161.29 205.74)
 		)
@@
 	(wire
 		(pts
-			(xy 129.54 220.98) (xy 132.08 220.98)
-		)
-		(stroke
-			(width 0)
-			(type default)
-		)
-	)
-	(wire
-		(pts
 			(xy 96.52 77.47) (xy 106.68 77.47)
 		)
@@
 		)
 	)
-	(label "EN1"
-		(at 132.08 220.98 0)
-		(effects
-			(font
-				(size 1.27 1.27)
-			)
-			(justify left bottom)
-		)
-	)
 	(label "FOD"
 		(at 125.73 113.03 270)
@@
 		)
 	)
-	(label "EN1"
-		(at 147.32 92.71 0)
-		(effects
-			(font
-				(size 1.27 1.27)
-			)
-			(justify left bottom)
-		)
-	)
