File: SmartCard.kicad_pcb (KiCad board)
At the start: 4 copper layers, 30 x 40 mm, 69 parts, among them IC1 BQ51003YFPT, IC2 BQ25100YFPR, IC3 BQ298009RUGR, Q1 EFC3J018NUZTDG, U1 NRF54L15-QFAA-R, U2 TPS62840YBGR, Y1 ABM11W-25.0000MHZ-7-D1X-T3, Y2 ECS-.327-7-12-TR

Commit message: mostly done just a little more work
Parts:
- removed C37: 1uF, Capacitor_SMD:C_0402_1005Metric
- removed R12: 4.7M, Resistor_SMD:R_0402_1005Metric
- added J1: Conn_01x05, Connector_PinHeader_2.54mm:PinHeader_1x05_P2.54mm_Vertical, F.Cu at (144.5, 70.5)
- added TP2: 1V8, TestPoint:TestPoint_Pad_2.0x2.0mm, B.Cu at (166.2, 99.2)
- added TP4: VDD, TestPoint:TestPoint_Pad_2.0x2.0mm, B.Cu at (144.5, 85.0)
- added TP5: VBUS, TestPoint:TestPoint_Pad_2.0x2.0mm, B.Cu at (153.2, 98.3)
- C14: value 1.3nF -> 1nF
- C7: value 47pF -> 330pF
- IC1: value BQ51003YFPT -> BQ51013BRHLR; footprint SamacSys_Parts:BGA28C40P4X7_188X301X50 -> Package_DFN_QFN:Texas_VQFN-RHL-20
- L2: footprint Inductor_SMD:L_1206_3216Metric_Pad1.22x1.90mm_HandSolder -> Inductor_SMD:L_1812_4532Metric_Pad1.30x3.40mm_HandSolder
- R10: value 50m -> 100m; footprint Resistor_SMD:R_0603_1608Metric -> Resistor_SMD:R_0805_2012Metric
- R7: value 6k -> 6.04k
- Y1: value ABM11W-25.0000MHZ-7-D1X-T3 -> 32MHz
- moved C10 51.4 mm to (154.8, 87.8), turned to -90 degrees
- moved C8 45.5 mm to (157.0, 95.7), turned to 90 degrees
- moved C12 43.9 mm to (155.2, 86.3)
- moved C20 42.8 mm to (153.3, 95.6), turned to 180 degrees
- moved C11 42.1 mm to (155.7, 87.8), turned to -90 degrees
- moved C9 41.0 mm to (150.6, 96.6)
- moved C13 40.1 mm to (156.0, 95.7), turned to 90 degrees
- moved R3 39.6 mm to (158.0, 85.6), turned to -90 degrees
- moved R2 37.5 mm to (158.5, 87.2)
- moved C21 37.3 mm to (152.8, 88.2), turned to 180 degrees
- moved C17 36.3 mm to (153.2, 96.8), turned to 180 degrees
- moved R1 34.8 mm to (158.0, 88.7), turned to -90 degrees
- moved R5 32.0 mm to (159.0, 88.6), turned to 90 degrees
- moved C18 31.9 mm to (152.5, 87.0), turned to 180 degrees
- moved E1 30.3 mm to (166.0, 90.3), turned to -90 degrees
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- renumbered R14 to R13
Connections:
- C10 pad 1: Net-(C10-Pad1) -> Net-(IC1-AC2)
- C11 pad 1: Net-(C10-Pad1) -> Net-(IC1-AC2)
- C12 pad 1: Net-(C10-Pad1) -> Net-(IC1-AC2)
- C12 pad 2: Net-(IC1-CLAMP1) -> Net-(IC1-CLAMP2)
- C13 pad 1: Net-(C13-Pad1) -> Net-(IC1-AC1)
- C13 pad 2: Net-(IC1-CLAMP2) -> Net-(IC1-CLAMP1)
- C14 pad 1: Net-(C13-Pad1) -> Net-(IC1-AC1)
- C14 pad 2: Net-(C10-Pad1) -> Net-(IC1-AC2)
- C5 pad 2: Net-(C13-Pad1) -> Net-(IC1-AC1)
- C6 pad 2: Net-(C13-Pad1) -> Net-(IC1-AC1)
- C7 pad 1: Net-(C13-Pad1) -> Net-(IC1-AC1)
- C7 pad 2: Net-(C10-Pad1) -> Net-(IC1-AC2)
- C8 pad 1: Net-(C13-Pad1) -> Net-(IC1-AC1)
- C9 pad 1: Net-(C13-Pad1) -> Net-(IC1-AC1)
- IC3 pad 5: /CTR -> -BATT
- L2 pad 1: Net-(C10-Pad1) -> Net-(IC1-AC2)
- R5 pad 1: Net-(IC1-TS-CTRL) -> Net-(IC1-TS/CTRL)
- U1 pad 13: unconnected-(U1-P2.02-Pad13) -> /EN1
- Y2 pad 1: (no net) -> /XL1
Routing:
- net VDD: track 0.00 -> 24.3 mm, vias 0 -> 8
- net /SWDCLK: track 0.00 -> 23.3 mm, vias 0 -> 1
- net /SWDIO: track 0.00 -> 22.8 mm, vias 0 -> 1
- net /RESET: track 0.00 -> 20.8 mm, vias 0 -> 1
- net /EN1: track 0.00 -> 16.0 mm, vias 0 -> 2
- net -BATT: track 0.00 -> 12.2 mm, vias 0 -> 4
- net GND: track 0.00 -> 11.4 mm, vias 0 -> 105
- net Net-(U1-DECA): track 0.00 -> 10.1 mm, vias 0 -> 3
- net Net-(C35-Pad2): track 0.00 -> 9.22 mm
- net /RECT: track 0.00 -> 8.32 mm
- net +1V8: track 0.00 -> 8.04 mm, vias 0 -> 8
- net Net-(IC1-AC2): track 0.00 -> 8.02 mm, vias 0 -> 4
- net Net-(IC1-AC1): track 0.00 -> 7.45 mm, vias 0 -> 3
- net Net-(IC3-DSG): track 0.00 -> 7.12 mm, vias 0 -> 2
- net Net-(IC1-CLAMP2): track 0.00 -> 7.00 mm, vias 0 -> 2
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- added copper zone on F.Cu, net +1V8
- added copper zone on In2.Cu, net +1V8
- added copper zone on B.Cu, net +BATT
- added copper zone on F.Cu, net +BATT
- added copper zone on B.Cu, net -BATT
- added copper zone on F.Cu, net -BATT
- added copper zone on F.Cu, net /RECT
- added copper zone on B.Cu, net GND
- added copper zone on F.Cu, net GND
- added copper zone on In1.Cu, net GND
- added copper zone on F.Cu, net Net-(C5-Pad1)
- added copper zone on F.Cu, net Net-(IC1-AC1)
- added copper zone on F.Cu, net Net-(IC1-AC2)
- added copper zone on F.Cu, net Net-(U1-DECA)
- added copper zone on F.Cu, net Net-(U1-DECD)
- added copper zone on F.Cu, net Net-(U2-SW)
- added copper zone on F.Cu, net VBUS
- added copper zone on F.Cu, net VDD
- added copper zone on In2.Cu, net VDD
Other:
- board size 30 x 40 mm -> 28 x 45 mm
- board text added: "+BATT"
- board text added: "-BATT"
- board text added: "1v8"
- board text added: "ANT"
- board text added: "GND"
- board text added: "RST"
- board text added: "RX"
- board text added: "SMART CARD"
- board text added: "SWDCLK"
- board text added: "SWDIO"
- board text added: "VDD"
- board text added: "nRF54L15"

Commit message: Added stitching vias
Routing:
- net GND: vias 105 -> 157

Commit message: Smart Card r2 done
Routing:
- net GND: vias 157 -> 155
Changed lines of the file:
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@@
 		(capping no)
 		(filling no)
+		(zone_defaults)
 		(grid_origin 141 67)
 		(pcbplotparams
@@
 		(sheetname "/")
 		(sheetfile "SmartCard.kicad_sch")
-		(units
-			(unit
-				(name "A")
-				(pins "2" "1")
-			)
-		)
 		(attr smd)
 		(duplicate_pad_numbers_are_jumpers no)
@@
 		)
 		(fp_line
-			(start -1.8 -0.2)
-			(end -1.8 -0.2)
+			(start -1.55 0)
+			(end -1.55 0)
 			(stroke
 				(width 0.1)
@@
 		)
 		(fp_line
-			(start -1.7 -0.2)
-			(end -1.7 -0.2)
+			(start -1.45 0)
+			(end -1.45 0)
 			(stroke
 				(width 0.1)
@@
 		)
 		(fp_arc
-			(start -1.8 -0.2)
-			(mid -1.75 -0.25)
-			(end -1.7 -0.2)
+			(start -1.55 0)
+			(mid -1.5 -0.05)
+			(end -1.45 0)
 			(stroke
 				(width 0.1)
@@
 		)
 		(fp_arc
-			(start -1.7 -0.2)
-			(mid -1.75 -0.15)
-			(end -1.8 -0.2)
+			(start -1.45 0)
+			(mid -1.5 0.05)
+			(end -1.55 0)
 			(stroke
 				(width 0.1)
@@
 	)
 	(via
-		(at 167.25 79.25)
-		(size 0.7)
-		(drill 0.3)
-		(layers "F.Cu" "B.Cu")
-		(free yes)
-		(net "GND")
-	)
-	(via
 		(at 148.1 72.5)
 		(size 0.7)
@@
 	)
 	(via
+		(at 148.7 88.75)
+		(size 0.45)
+		(drill 0.2)
+		(layers "F.Cu" "B.Cu")
+		(free yes)
+		(net "GND")
+	)
+	(via
 		(at 151 106)
 		(size 0.7)
@@
 	)
 	(via
-		(at 164.35 85.85)
-		(size 0.7)
-		(drill 0.3)
-		(layers "F.Cu" "B.Cu")
-		(free yes)
-		(net "GND")
-	)
-	(via
 		(at 159 106)
 		(size 0.7)
@@
 	)
 	(via
-		(at 167.25 82.25)
+		(at 148 111)
 		(size 0.7)
 		(drill 0.3)
@@
 	)
 	(via
-		(at 148 111)
+		(at 167.25 83.65)
 		(size 0.7)
 		(drill 0.3)
@@
 	)
 	(via
-		(at 167.25 83.65)
+		(at 153.5 92.5)
 		(size 0.7)
 		(drill 0.3)
 		(layers "F.Cu" "B.Cu")
-		(free yes)
 		(net "GND")
 	)
 	(via
-		(at 153.5 92.5)
-		(size 0.7)
-		(drill 0.3)
+		(at 151.35 88.25)
+		(size 0.45)
+		(drill 0.2)
 		(layers "F.Cu" "B.Cu")
+		(free yes)
 		(net "GND")
 	)
@@
 	)
 	(via
-		(at 167.25 78.25)
-		(size 0.7)
-		(drill 0.3)
-		(layers "F.Cu" "B.Cu")
-		(free yes)
-		(net "GND")
-	)
-	(via
 		(at 164.75 79.25)
 		(size 0.7)
@@
 		(start 165 76.8)
 		(end 164.6 76.8)
-		(width 0.4)
+		(width 0.3058)
 		(layer "F.Cu")
 		(net "Net-(C35-Pad2)")
@@
 		(start 166 77.8)
 		(end 165 76.8)
-		(width 0.4)
+		(width 0.3058)
 		(layer "F.Cu")
 		(net "Net-(C35-Pad2)")
@@
 		(start 166 83.65)
 		(end 166 77.8)
-		(width 0.4)
+		(width 0.3058)
 		(layer "F.Cu")
 		(net "Net-(C35-Pad2)")
@@
 		(layer "F.Cu")
 		(hatch edge 0.5)
-		(priority 17)
+		(priority 18)
 		(connect_pads yes
 			(clearance 0.1)
@@
 		(layer "F.Cu")
 		(hatch edge 0.5)
-		(priority 28)
+		(priority 32)
 		(connect_pads yes
 			(clearance 0.2)
@@
 		(polygon
 			(pts
-				(xy 163.3 76.1) (xy 164.15 76.1) (xy 164.45 76.4) (xy 164.75 76.4) (xy 165.05 76.1) (xy 165.45 76.1)
-				(xy 165.45 75.6) (xy 165.2 75.35) (xy 163.95 75.35) (xy 163.3 76)
+				(xy 163.3 76.1) (xy 164.15 76.1) (xy 164.45 76.4) (xy 164.75 76.4) (xy 165.35 76.4) (xy 165.45 76.1)
+				(xy 165.45 75.6) (xy 165.2 75.35) (xy 163.3 75.35)
 			)
 		)
@@
 		(layer "F.Cu")
 		(hatch edge 0.5)
-		(priority 18)
+		(priority 19)
 		(connect_pads yes
 			(clearance 0.2)
@@
 	)
 	(zone
+		(net "GND")
+		(layer "F.Cu")
+		(hatch edge 0.5)
+		(priority 34)
+		(connect_pads yes
+			(clearance 0.2)
+		)
+		(min_thickness 0.25)
+		(fill yes
+			(thermal_gap 0.5)
+			(thermal_bridge_width 0.5)
+			(island_removal_mode 0)
+		)
+		(polygon
+			(pts
+				(xy 165.05 77.55) (xy 165.05 76.1) (xy 165.3 75.85) (xy 165.6 75.85) (xy 168.59826 75.849314) (xy 168.6 83.45)
+				(xy 166.8 83.45) (xy 166.35 83) (xy 164.85 83) (xy 164.65 82.8) (xy 164.65 77.55)
+			)
+		)
+	)
+	(zone
 		(net "Net-(IC1-AC2)")
 		(layer "F.Cu")
@@
 		(layer "F.Cu")
 		(hatch edge 0.5)
-		(priority 12)
+		(priority 13)
 		(connect_pads yes
-			(clearance 0.5)
+			(clearance 0.3)
 		)
 		(min_thickness 0.25)
@@
 		(layer "F.Cu")
 		(hatch edge 0.5)
-		(priority 31)
+		(priority 29)
 		(connect_pads yes
 			(clearance 0.2)
@@
 		(layer "F.Cu")
 		(hatch edge 0.5)
-		(priority 32)
+		(priority 27)
 		(connect_pads yes
 			(clearance 0)
@@
 		(layer "F.Cu")
 		(hatch edge 0.5)
-		(priority 29)
+		(priority 31)
 		(connect_pads yes
 			(clearance 0.5)
@@
 		(layer "F.Cu")
 		(hatch edge 0.5)
-		(priority 19)
+		(priority 20)
 		(connect_pads yes
 			(clearance 0.5)
@@
 		(layer "F.Cu")
 		(hatch edge 0.5)
+		(priority 28)
+		(connect_pads
+			(clearance 0.3)
+		)
+		(min_thickness 0.25)
+		(fill yes
+			(thermal_gap 0.5)
+			(thermal_bridge_width 0.5)
+			(island_removal_mode 0)
+		)
+		(polygon
+			(pts
+				(xy 152.45 87.95) (xy 151.3 87.95) (xy 151.05 88.2) (xy 151.05 88.6) (xy 151.65 89.2) (xy 152.4 89.2)
+				(xy 152.55 89.05) (xy 152.55 88.05)
+			)
+		)
+	)
+	(zone
+		(net "GND")
+		(layer "F.Cu")
+		(hatch edge 0.5)
 		(priority 30)
 		(connect_pads yes
@@
 		(layer "F.Cu")
 		(hatch edge 0.5)
-		(priority 14)
+		(priority 15)
 		(connect_pads yes
 			(clearance 0.1)
@@
 		(layer "F.Cu")
 		(hatch edge 0.5)
-		(priority 15)
+		(priority 16)
 		(connect_pads yes
 			(clearance 0.5)
@@
 		(layer "F.Cu")
 		(hatch edge 0.5)
-		(priority 27)
+		(priority 33)
 		(connect_pads yes
 			(clearance 0.3)
@@
 		(layer "F.Cu")
 		(hatch edge 0.5)
-		(priority 16)
+		(priority 17)
 		(connect_pads yes
 			(clearance 0.1)
@@
 		(layer "F.Cu")
 		(hatch edge 0.5)
-		(priority 13)
+		(priority 14)
 		(connect_pads yes
 			(clearance 0.5)
@@
 		(layers "F.Cu" "B.Cu" "In1.Cu")
 		(hatch edge 0.5)
-		(priority 2)
 		(connect_pads
 			(clearance 0.5)
@@
 		(polygon
 			(pts
-				(xy 141 67) (xy 169 67) (xy 169 112) (xy 141 112)
+				(xy 169 112) (xy 141 112) (xy 141 67) (xy 169 67)
 			)
 		)
@@
 		(polygon
 			(pts
-				(xy 159.35 75.7) (xy 163.75 75.7) (xy 164.45 76.4) (xy 164.75 76.4) (xy 165.05 76.1) (xy 165.05 77.55)
+				(xy 159.35 75.7) (xy 163.75 75.7) (xy 164.45 76.4) (xy 164.75 76.4) (xy 165.05 76.4) (xy 165.05 77.55)
 				(xy 159.65 77.55) (xy 159.35 77.25)
 			)
@@
 		(layer "B.Cu")
 		(hatch edge 0.5)
-		(priority 1)
+		(priority 2)
 		(connect_pads yes
 			(clearance 0.5)
@@
 		(layer "B.Cu")
 		(hatch edge 0.5)
-		(priority 11)
+		(priority 12)
 		(connect_pads yes
 			(clearance 0.5)
@@
 		(layer "B.Cu")
 		(hatch edge 0.5)
+		(priority 1)
 		(connect_pads yes
 			(clearance 0.5)

Commit message: finished pack swap
Parts:
- C7: value 330pF -> 100pF
- moved TP5 0.32 mm to (153.4, 98.1)
- turned R10 to 0 degrees
Connections:
- C32 pad 2: GND -> -BATT
- IC1 pad 10: /EN1 -> GND
- IC3 pad 3: GND -> -BATT
- IC3 pad 4: -BATT -> GND
- IC3 pad 5: -BATT -> GND
- Q1 pad 2: Net-(IC3-CHG) -> Net-(IC3-DSG)
- Q1 pad 5: Net-(IC3-DSG) -> Net-(IC3-CHG)
- R10 pad 1: GND -> -BATT
- R10 pad 2: -BATT -> GND
- R11 pad 1: VDD -> +BATT
- R13 pad 1: +BATT -> VDD
- R9 pad 1: VDD -> +BATT
- U1 pad 13: /EN1 -> unconnected-(U1-P2.02-Pad13)
Routing:
- net /EN1: track 16.0 -> 0.00 mm, vias 2 -> 0
- net +BATT: track 4.82 -> 12.3 mm, vias 3 -> 4
- net Net-(IC3-DSG): track 7.12 -> 5.20 mm, vias 2 -> 0
- net Net-(IC3-CHG): track 5.00 -> 6.90 mm, vias 0 -> 2
- net GND: track 11.4 -> 12.6 mm
- net -BATT: track 12.2 -> 13.3 mm, vias 4 -> 5
- net VDD: track 24.3 -> 25.3 mm, vias 8 -> 6
